Commit message: Stabilize supervised 13-view scan pipeline

File: piper_ros_foxy/src/piper_description/urdf/piper_description.xacro (robot description, xacro)
@@ -1,6 +1,4 @@
 <?xml version="1.0" encoding="utf-8"?>
-<robot
-  name="arm"
-  xmlns:xacro="http://ros.org/wiki/xacro">
+<robot name="arm">
 <!-- world -->
   <link name="world"/>
@@ -124,8 +122,9 @@
     name="joint2"
     type="revolute">
+    <!-- Mode-0 controller/FK offset. Do not add the optional SDK mode-1
+         two-degree J2/J3 correction to the robot_state_publisher model. -->
     <origin
       xyz="0 0 0"
-      rpy="1.5708 -0.1359 -3.1416" />
-      <!-- rpy="1.5708 -0.10095-0.03490659 -3.1416" /> -->
+      rpy="1.5707963267948966 -0.10088003076527219 -3.141592653589793" />
     <parent
       link="link1" />
@@ -134,6 +133,9 @@
     <axis
       xyz="0 0 1" />
-    <limit
-      lower="0"
+    <!-- Existing validated controller-coordinate bound from
+         piper_joint_bounds.json. This small negative range is required for
+         the reported mode-0 zero state; it is not a new measurement. -->
+    <limit
+      lower="-0.044796192"
       upper="3.14"
       effort="100"
@@ -176,6 +178,5 @@
     <origin
       xyz="0.28503 0 0"
-      rpy="0 0 -1.7939" />
-      <!-- rpy="0 0 -1.759-0.03490659" /> -->
+      rpy="0 0 -1.7589428201598853" />
     <parent
       link="link2" />
@@ -225,6 +226,6 @@
     type="revolute">
     <origin
-      xyz="-0.021984 -0.25075 0"
-      rpy="1.5708 0 0" />
+      xyz="-0.02198 -0.25075 0"
+      rpy="1.5707963267948966 0 0" />
     <parent
       link="link3" />
@@ -275,5 +276,5 @@
     <origin
       xyz="0 0 0"
-      rpy="-1.5708 0 0" />
+      rpy="-1.5707963267948966 0 0" />
     <parent
       link="link4" />
@@ -323,6 +324,6 @@
     type="revolute">
     <origin
-      xyz="8.8259E-05 -0.091 0"
-      rpy="1.5708 0 0" />
+      xyz="0 -0.091 0"
+      rpy="1.5707963267948966 0 0" />
     <parent
       link="link5" />
@@ -504,58 +505,3 @@
       velocity="1" />
   </joint>
-<!-- controller -->
-  <xacro:macro name="transmission_block" params="tran_name joint_name motor_name">
-    <transmission name="${tran_name}">
-        <type>transmission_interface/SimpleTransmission</type>
-        <joint name="${joint_name}">
-            <hardwareInterface>hardware_interface/PositionJointInterface</hardwareInterface>
-        </joint>
-        <actuator name="$motor_name">
-            <hardwareInterface>hardware_interface/PositionJointInterface</hardwareInterface>
-            <mechanicalReduction>1</mechanicalReduction>
-        </actuator>
-    </transmission>
-  </xacro:macro>
-  <xacro:transmission_block tran_name="tran1" joint_name="joint1" motor_name="motor1"/>
-  <xacro:transmission_block tran_name="tran2" joint_name="joint2" motor_name="motor2"/>
-  <xacro:transmission_block tran_name="tran3" joint_name="joint3" motor_name="motor3"/>
-  <xacro:transmission_block tran_name="tran4" joint_name="joint4" motor_name="motor4"/>
-  <xacro:transmission_block tran_name="tran5" joint_name="joint5" motor_name="motor5"/>
-  <xacro:transmission_block tran_name="tran6" joint_name="joint6" motor_name="motor6"/>
-  <xacro:transmission_block tran_name="tran7" joint_name="joint7" motor_name="motor7"/>
-  <xacro:transmission_block tran_name="tran8" joint_name="joint8" motor_name="motor8"/>
-<!-- gazebo -->
-  <gazebo>
-    <plugin name="gazebo_ros_control" filename="libgazebo_ros_control.so">
-        <robotNamespace>/piper_description</robotNamespace>
-        <legacyModeNS>true</legacyModeNS>
-    </plugin>
-  </gazebo>
-  <gazebo reference="base_link">
-    <material>Gazebo/Black</material>
-  </gazebo>
-  <gazebo reference="link1">
-    <material>Gazebo/White</material>
-  </gazebo>
-  <gazebo reference="link2">
-    <material>Gazebo/White</material>
-  </gazebo>
-  <gazebo reference="link3">
-    <material>Gazebo/White</material>
-  </gazebo>
-  <gazebo reference="link4">
-    <material>Gazebo/Black</material>
-  </gazebo>
-  <gazebo reference="link5">
-    <material>Gazebo/White</material>
-  </gazebo>
-  <gazebo reference="link6">
-    <material>Gazebo/White</material>
-  </gazebo>
-  <gazebo reference="link7">
-    <material>Gazebo/Orange</material>
-  </gazebo>
-  <gazebo reference="link8">
-    <material>Gazebo/Orange</material>
-  </gazebo>
 </robot>

Commit message: feat: integrate platform capability map and ray seed repair

File: piper_ros_foxy/src/piper_description/urdf/piper_description.xacro (robot description, xacro)
@@ -39,4 +39,43 @@
     </collision>
   </link>
+  <!--
+    The tracked platform is a permanent part of the installed assembly.  The
+    source meshes below are already transformed into base_link coordinates, so
+    their fixed joints are identities.  These links are visual-only here;
+    model_builder.py installs the hash-verified decomposed collision pieces for
+    Tesseract without creating a second platform representation.
+  -->
+  <link name="bunker_chassis_collision">
+    <visual>
+      <origin xyz="0 0 0" rpy="0 0 0" />
+      <geometry>
+        <mesh filename="package://piper_description/meshes/bunker_chassis_collision.STL" />
+      </geometry>
+      <material name="bunker_dark">
+        <color rgba="0.16 0.18 0.20 1" />
+      </material>
+    </visual>
+  </link>
+  <joint name="base_link_to_bunker_chassis_collision" type="fixed">
+    <origin xyz="0 0 0" rpy="0 0 0" />
+    <parent link="base_link" />
+    <child link="bunker_chassis_collision" />
+  </joint>
+  <link name="bunker_sensor_station_collision">
+    <visual>
+      <origin xyz="0 0 0" rpy="0 0 0" />
+      <geometry>
+        <mesh filename="package://piper_description/meshes/bunker_sensor_station_collision.STL" />
+      </geometry>
+      <material name="bunker_station">
+        <color rgba="0.28 0.34 0.40 1" />
+      </material>
+    </visual>
+  </link>
+  <joint name="base_link_to_bunker_sensor_station_collision" type="fixed">
+    <origin xyz="0 0 0" rpy="0 0 0" />
+    <parent link="base_link" />
+    <child link="bunker_sensor_station_collision" />
+  </joint>
   <link
     name="link1">
