Commit message: Correct symmetric J1 limits and ray review state

File: integration/track_robot_description/drop_in/src/bunker_pro2/urdf/bunker_pro2.urdf (robot description, URDF)
Before this commit: robot bunker_pro2, 19 links, 18 joints
Joints:
- joint joint1: limit lower=-2.618 upper=2.168 effort=100 velocity=5 -> lower=-2.6179 upper=2.6179 effort=100 velocity=5

File: integration/track_robot_description/drop_in/src/piper_description/urdf/piper_description.xacro (robot description, xacro)
@@ -55,5 +55,5 @@
     <child link="link1" />
     <axis xyz="0 0 1" />
-    <limit lower="-2.618" upper="2.168" effort="100" velocity="5" />
+    <limit lower="-2.6179" upper="2.6179" effort="100" velocity="5" />
   </joint>
   <link name="link2">

File: piper_ros_foxy/src/piper_description/urdf/piper_description.urdf (robot description, URDF)
Before this commit: robot piper_description, 10 links, 9 joints
Joints:
- joint joint1: limit lower=-2.618 upper=2.168 effort=100 velocity=5 -> lower=-2.6179 upper=2.6179 effort=100 velocity=5

File: piper_ros_foxy/src/piper_description/urdf/piper_description.xacro (robot description, xacro)
@@ -122,6 +122,6 @@
       xyz="0 0 1" />
     <limit
-      lower="-2.618"
-      upper="2.168"
+      lower="-2.6179"
+      upper="2.6179"
       effort="100"
       velocity="5" />
